Commit message: Dummy base_link inertia

File: urdf/talos_full_v2.urdf (robot description, URDF)
Before this commit: robot talos, 60 links, 59 joints
Links:
- added link base_inertia_dummy, mass 15.36284
- link base_link: mass 15.36284 -> None
Joints:
- added joint dummy_inertia_joint: type fixed, parent base_link, child base_inertia_dummy, origin xyz=0.0 0 0.0 rpy=0 0 0
